File: kicad/ESPonics/ESPonics.kicad_sch (KiCad schematic)
At the start: 8 parts, among them J1 RJ45, J2 RJ45, J3 RJ45, J4 Conn_01x02_Pin, U1 ESP32-DevKitC

Commit message: Small pcb changes
Parts:
- added J5: Conn_01x02_Pin, Connector_JST:JST_XH_B2B-XH-A_1x02_P2.50mm_Vertical, symbol Connector:Conn_01x02_Pin
- J2: footprint (none) -> Connector_RJ:RJ45_Amphenol_54602-x08_Horizontal
- R1: footprint (none) -> Resistor_THT:R_Axial_DIN0204_L3.6mm_D1.6mm_P1.90mm_Vertical
- U1: footprint Espressif:ESP32-DevKitC -> PCM_Espressif:ESP32-DevKitC
Connections:
- net GND: now also J5.2 (Pin_2)
- net at U1.2 (CHIP_PU): now also J5.1 (Pin_1)
Changed lines of the file:
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@@
   (junction (at 93.98 68.58) (diameter 0) (color 0 0 0 0)
   )
+  (junction (at 80.01 151.13) (diameter 0) (color 0 0 0 0)
+  )
   (junction (at 38.1 106.68) (diameter 0) (color 0 0 0 0)
   )
@@
     (stroke (width 0) (type default))
   )
+  (wire (pts (xy 171.45 55.88) (xy 176.53 55.88))
+    (stroke (width 0) (type default))
+  )
   (wire (pts (xy 69.85 76.2) (xy 69.85 71.12))
     (stroke (width 0) (type default))
@@
     (stroke (width 0) (type default))
   )
+  (wire (pts (xy 80.01 151.13) (xy 151.13 151.13))
+    (stroke (width 0) (type default))
+  )
+  (wire (pts (xy 66.04 29.21) (xy 171.45 29.21))
+    (stroke (width 0) (type default))
+  )
   (wire (pts (xy 29.21 26.67) (xy 29.21 148.59))
     (stroke (width 0) (type default))
@@
     (stroke (width 0) (type default))
   )
-  (wire (pts (xy 35.56 151.13) (xy 151.13 151.13))
+  (wire (pts (xy 35.56 151.13) (xy 80.01 151.13))
     (stroke (width 0) (type default))
   )
@@
     (stroke (width 0) (type default))
   )
+  (wire (pts (xy 80.01 31.75) (xy 80.01 151.13))
+    (stroke (width 0) (type default))
+  )
   (wire (pts (xy 176.53 63.5) (xy 151.13 63.5))
     (stroke (width 0) (type default))
@@
     (stroke (width 0) (type default))
   )
+  (wire (pts (xy 171.45 29.21) (xy 171.45 55.88))
+    (stroke (width 0) (type default))
+  )
   (wire (pts (xy 176.53 76.2) (xy 158.75 76.2))
     (stroke (width 0) (type default))
@@
     (stroke (width 0) (type default))
   )
+  (wire (pts (xy 66.04 31.75) (xy 80.01 31.75))
+    (stroke (width 0) (type default))
+  )
   (wire (pts (xy 64.77 100.33) (xy 173.99 100.33))
     (stroke (width 0) (type default))
@@
         (path "/c3daf4c9-5e4c-4393-8644-666075c44fa8"
           (reference "R3") (unit 1)
+        )
+      )
+    )
+  )
+  (symbol (lib_id "Connector:Conn_01x02_Pin") (at 60.96 29.21 0) (unit 1)
+    (in_bom yes) (on_board yes) (dnp no) (fields_autoplaced)
+    (property "Reference" "J5" (at 61.595 24.13 0)
+      (effects (font (size 1.27 1.27)))
+    )
+    (property "Value" "Conn_01x02_Pin" (at 61.595 26.67 0)
+      (effects (font (size 1.27 1.27)))
+    )
+    (property "Footprint" "Connector_JST:JST_XH_B2B-XH-A_1x02_P2.50mm_Vertical" (at 60.96 29.21 0)
+      (effects (font (size 1.27 1.27)) hide)
+    )
+    (property "Datasheet" "~" (at 60.96 29.21 0)
+      (effects (font (size 1.27 1.27)) hide)
+    )
+    (pin "1")
+    (pin "2")
+    (instances
+      (project "ESPonics"
+        (path "/c3daf4c9-5e4c-4393-8644-666075c44fa8"
+          (reference "J5") (unit 1)
         )
       )
@@
       (effects (font (size 1.27 1.27)))
     )
-    (property "Footprint" "" (at 54.61 94.615 90)
+    (property "Footprint" "Connector_RJ:RJ45_Amphenol_54602-x08_Horizontal" (at 54.61 94.615 90)
       (effects (font (size 1.27 1.27)) hide)
     )
@@
       (effects (font (size 1.27 1.27)) (justify left))
     )
-    (property "Footprint" "" (at 149.352 139.7 90)
+    (property "Footprint" "Resistor_THT:R_Axial_DIN0204_L3.6mm_D1.6mm_P1.90mm_Vertical" (at 149.352 139.7 90)
       (effects (font (size 1.27 1.27)) hide)
     )
@@
       (effects (font (size 1.27 1.27)) (justify left))
     )
-    (property "Footprint" "Espressif:ESP32-DevKitC" (at 209.55 129.54 0)
-      (effects (font (size 1.27 1.27)))
-    )
+    (property "Footprint" "PCM_Espressif:ESP32-DevKitC" (at 209.55 129.54 0)
+      (effects (font (size 1.27 1.27)))
+    )

Commit message: Update schematic with new GPIOs
Connections:
- net at J1.3, R3.2: now also U1.10 (DAC_2/ADC2_CH9/GPIO26); no longer U1.3 (SENSOR_VP/GPIO36/ADC1_CH0)
- net at J1.2, R2.2: no longer U1.4 (SENSOR_VN/GPIO39/ADC1_CH3)
Changed lines of the file:
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@@
-    (stroke (width 0) (type default))
-  )
-  (wire (pts (xy 176.53 86.36) (xy 143.51 86.36))
     (stroke (width 0) (type default))
   )
@@
     (stroke (width 0) (type default))
   )
+  (wire (pts (xy 143.51 34.29) (xy 260.35 34.29))
+    (stroke (width 0) (type default))
+  )
   (wire (pts (xy 176.53 73.66) (xy 156.21 73.66))
     (stroke (width 0) (type default))
   )
+  (wire (pts (xy 143.51 66.04) (xy 143.51 34.29))
+    (stroke (width 0) (type default))
+  )
   (wire (pts (xy 153.67 92.71) (xy 153.67 71.12))
     (stroke (width 0) (type default))
   )
+  (wire (pts (xy 260.35 88.9) (xy 242.57 88.9))
+    (stroke (width 0) (type default))
+  )
   (wire (pts (xy 73.66 121.92) (xy 64.77 121.92))
     (stroke (width 0) (type default))
@@
     (stroke (width 0) (type default))
   )
-  (wire (pts (xy 140.97 88.9) (xy 140.97 68.58))
-    (stroke (width 0) (type default))
-  )
   (wire (pts (xy 93.98 68.58) (xy 140.97 68.58))
     (stroke (width 0) (type default))
@@
     (stroke (width 0) (type default))
   )
-  (wire (pts (xy 176.53 88.9) (xy 140.97 88.9))
-    (stroke (width 0) (type default))
-  )
   (wire (pts (xy 176.53 97.79) (xy 176.53 124.46))
     (stroke (width 0) (type default))
@@
     (stroke (width 0) (type default))
   )
+  (wire (pts (xy 260.35 34.29) (xy 260.35 88.9))
+    (stroke (width 0) (type default))
+  )
   (wire (pts (xy 29.21 25.4) (xy 29.21 26.67))
     (stroke (width 0) (type default))
@@
     (stroke (width 0) (type default))
   )
-  (wire (pts (xy 143.51 66.04) (xy 143.51 86.36))
-    (stroke (width 0) (type default))
-  )

Commit message: Update kicad file
Connections:
- net at J1.2, R2.2: now also U1.8 (32K_XN/GPIO33/ADC1_CH5)
- net at U1.3 (SENSOR_VP/GPIO36/ADC1_CH0): now also J1.5
- net at U1.4 (SENSOR_VN/GPIO39/ADC1_CH3): now also J1.6
- net at U1.5 (VDET_1/GPIO34/ADC1_CH6): no longer J1.5
Changed lines of the file:
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@@
-    (stroke (width 0) (type default))
-  )
-  (wire (pts (xy 151.13 63.5) (xy 151.13 58.42))
     (stroke (width 0) (type default))
   )
@@
     (stroke (width 0) (type default))
   )
+  (wire (pts (xy 161.29 88.9) (xy 176.53 88.9))
+    (stroke (width 0) (type default))
+  )
   (wire (pts (xy 212.09 45.72) (xy 212.09 48.26))
     (stroke (width 0) (type default))
@@
     (stroke (width 0) (type default))
   )
+  (wire (pts (xy 151.13 68.58) (xy 151.13 129.54))
+    (stroke (width 0) (type default))
+  )
   (wire (pts (xy 29.21 151.13) (xy 35.56 151.13))
     (stroke (width 0) (type default))
   )
+  (wire (pts (xy 163.83 86.36) (xy 176.53 86.36))
+    (stroke (width 0) (type default))
+  )
   (wire (pts (xy 64.77 87.63) (xy 101.6 87.63))
     (stroke (width 0) (type default))
   )
-  (wire (pts (xy 151.13 58.42) (xy 64.77 58.42))
+  (wire (pts (xy 64.77 58.42) (xy 161.29 58.42))
     (stroke (width 0) (type default))
   )
@@
     (stroke (width 0) (type default))
   )
+  (wire (pts (xy 163.83 60.96) (xy 163.83 86.36))
+    (stroke (width 0) (type default))
+  )
   (wire (pts (xy 66.04 29.21) (xy 171.45 29.21))
     (stroke (width 0) (type default))
@@
     (stroke (width 0) (type default))
   )
-  (wire (pts (xy 176.53 81.28) (xy 148.59 81.28))
+  (wire (pts (xy 161.29 58.42) (xy 161.29 88.9))
     (stroke (width 0) (type default))
   )
@@
     (stroke (width 0) (type default))
   )
-  (wire (pts (xy 151.13 68.58) (xy 151.13 129.54))
-    (stroke (width 0) (type default))
-  )
   (wire (pts (xy 71.12 102.87) (xy 71.12 106.68))
     (stroke (width 0) (type default))
@@
     (stroke (width 0) (type default))
   )
-  (wire (pts (xy 148.59 81.28) (xy 148.59 60.96))
-    (stroke (width 0) (type default))
-  )
   (wire (pts (xy 93.98 45.72) (xy 38.1 45.72))
     (stroke (width 0) (type default))
@@
     (stroke (width 0) (type default))
   )
-  (wire (pts (xy 93.98 68.58) (xy 140.97 68.58))
+  (wire (pts (xy 93.98 68.58) (xy 148.59 68.58))
     (stroke (width 0) (type default))
   )
@@
     (stroke (width 0) (type default))
   )
-  (wire (pts (xy 176.53 63.5) (xy 151.13 63.5))
-    (stroke (width 0) (type default))
-  )
   (wire (pts (xy 176.53 97.79) (xy 176.53 124.46))
     (stroke (width 0) (type default))
@@
     (stroke (width 0) (type default))
   )
+  (wire (pts (xy 148.59 63.5) (xy 176.53 63.5))
+    (stroke (width 0) (type default))
+  )
   (wire (pts (xy 260.35 34.29) (xy 260.35 88.9))
     (stroke (width 0) (type default))
@@
     (stroke (width 0) (type default))
   )
-  (wire (pts (xy 64.77 60.96) (xy 148.59 60.96))
+  (wire (pts (xy 64.77 60.96) (xy 163.83 60.96))
     (stroke (width 0) (type default))
   )
@@
     (stroke (width 0) (type default))
   )
+  (wire (pts (xy 148.59 68.58) (xy 148.59 63.5))
+    (stroke (width 0) (type default))
+  )
